File: src/main/odroid_h3p.kicad_sch (KiCad schematic)
At the start: 2 parts, among them J301 Conn_02x12_Odd_Even, J302 Conn_01x12

Commit message: Additions and fixes:
Add:
- Add power rail LED status indicators
- Buffered LED on ETH_LINK
- GPIO14 and GPIO12 on header
- GPIO14 5V buffered output on header
- Testpoints for GPIO0 and ESP32_ENABLE pin
- Reset and Boot switches
- ESP PWR selector switch
- USB Type-C PD input (5V) for ESP32
- 1.1A Fuse for USB PD input
- Add spot for BIOS battery on silk
- Add silkscreen default jumper marking
- Add GPIO39 external pullup to 3V3
- Add pulldown to PWR_BUTTON (GPIO15)
- Add silkscreen github link

Fixes:
- Clarify things on silk
- Make pinout compatible with USB-UART boards
  - Move GPI0 and ENABLE to testpoints
- Silkscreen alignment fixes

Removed:
- 3 APA102 LEDs
- Remove JP201
Parts:
- added D101: 3V3_RUN, LED_SMD:LED_0603_1608Metric, symbol Device:LED
- added D103: 5V_RUN, LED_SMD:LED_0603_1608Metric, symbol Device:LED
- added D104: 5V_STBY, LED_SMD:LED_0603_1608Metric, symbol Device:LED
- added R105, R107, R108: 100R, Resistor_SMD:R_0402_1005Metric, symbol Device:R
Connections:
- net +3V3_RUN: now also R105.1
- net +5V_RUN: now also R107.1
- net +5V_STBY: now also R108.1
- net GND: now also D101.1 (K), D103.1 (K), D104.1 (K)
- new net: D101.2 (A), R105.2
- new net: D103.2 (A), R107.2
- new net: D104.2 (A), R108.2
