File: src/main/wt32_eth01.kicad_sch (KiCad schematic)
At the start: 14 parts, among them J101 Conn_01x10, J105 Conn_01x06, U101 CD74HCT125M96, U202 WT32-ETH01-M3

Commit message: Additions and fixes:
Add:
- Add power rail LED status indicators
- Buffered LED on ETH_LINK
- GPIO14 and GPIO12 on header
- GPIO14 5V buffered output on header
- Testpoints for GPIO0 and ESP32_ENABLE pin
- Reset and Boot switches
- ESP PWR selector switch
- USB Type-C PD input (5V) for ESP32
- 1.1A Fuse for USB PD input
- Add spot for BIOS battery on silk
- Add silkscreen default jumper marking
- Add GPIO39 external pullup to 3V3
- Add pulldown to PWR_BUTTON (GPIO15)
- Add silkscreen github link

Fixes:
- Clarify things on silk
- Make pinout compatible with USB-UART boards
  - Move GPI0 and ENABLE to testpoints
- Silkscreen alignment fixes

Removed:
- 3 APA102 LEDs
- Remove JP201
Parts:
- removed C204, C205, C206: 100nF, Capacitor_SMD:C_0402_1005Metric, symbol Device:C
- removed D101 (x3): APA102-2020, odroid_h3_uitx_adapter:LED-APA102-2020, symbol odroid_h3_uitx_adapter:APA102-2020
- removed JP101: Jumper_3_Open, Jumper:SolderJumper-3_P1.3mm_Open_RoundedPad1.0x1.5mm_NumberLabels, symbol Jumper:Jumper_3_Open
- added D102: ETH_LINK, LED_SMD:LED_0603_1608Metric, symbol Device:LED
- added D102: 3V3_ESP32, LED_SMD:LED_0603_1608Metric, symbol Device:LED
- added J501: Conn_01x03, odroid_h3_uitx_adapter:PinHeader_1x03_P2.54mm_Vertical, symbol odroid_h3_uitx_adapter:Conn_01x03
- added R101 (x2): 100K, Resistor_SMD:R_0402_1005Metric, symbol Device:R
- added R106 (x2): 100R, Resistor_SMD:R_0402_1005Metric, symbol Device:R
- added SW201, SW202: TS-1187A-B-A-B, easyeda2kicad:SW-SMD_4P-L5.1-W5.1-P3.70-LS6.5-TL-2, symbol easyeda2kicad:TS-1187A-B-A-B
- added TP201: ENABLE, TestPoint:TestPoint_Pad_D2.0mm, symbol Connector:TestPoint_Probe
- added TP202: GPI0, TestPoint:TestPoint_Pad_D2.0mm, symbol Connector:TestPoint_Probe
Connections:
- net LED_DATA_OUT is gone; now on net GPIO12: J101.9 (Pin_9)
- net LED_DAT_LV is gone; now on net GPIO14: U101.5, U202.19 (I/O14)
- net +3V3_ESP: now also J501.2 (Pin_2), R101.1, R106.1; no longer J105.6 (Pin_6)
- net ENABLE: now also TP201.1; no longer J105.5 (Pin_5)
- net ETH_LLINK: now also U101.2; no longer U101.12
- net GND: now also J101.3 (Pin_3), J105.6 (Pin_6), D102.1 (K), D102.1 (K), R101.2, SW201.3 (C), SW201.4 (D), SW202.3 (C), SW202.4 (D); no longer J101.7 (Pin_7), J105.1 (Pin_1)
- net GPI0: now also SW202.1 (A), SW202.2 (B), TP202.1; no longer J105.2 (Pin_2)
- net GPI39: now also R101.2
- net GPIO04: now also U101.12; no longer J101.3 (Pin_3)
- net PWR_ON_LV: now also R101.1
- net UART_PROG_TX: now also J105.2 (Pin_2); no longer J105.4 (Pin_4)
- net at U202.4 (EN1): now also SW201.1 (A), SW201.2 (B)
- net ETH_LINK renamed HDD_INDICATOR
- net LED_CLK_HV: no longer names the net of U101.3
- net LED_CLK_HV: now also R106.1
- net LED_CLK_LV renamed GPIO12
- net GPIO12: no longer U101.2
- net LED_CLOCK_OUT renamed GPIO14
- net LED_DAT_HV renamed GPIO14_5V
- net GPIO14_5V: now also J101.7 (Pin_7)
- new net: D102.2 (A), R106.2 (x2)
- new net: J105.4 (Pin_4), J501.3 (Pin_3)
- no-connect marks 1 -> 4
